File: main_board/main_board.kicad_sch (KiCad schematic)
At the start: 12 parts, among them J1 5V IN, J12 I2C ENV, J13 ENVPIR, J2 3.3V IN, J3 I2C PIR, J4 3.3V OUT, J5 3.3V OUT, J6 BH1750 (lux), J7 HDC1080 (temp&hum), U1 ESP32-S2-Saola-1

Commit message: Update to v0.5
Parts:
- removed U1: ESP32-S2-Saola-1, miro-v04:ESP32-S2-Saola-1, symbol main_board-rescue:ESP32-S2-Saola-1-miro-v04
- added U2: ESP32-S2-DevKitM, PCM_Espressif:ESP32-S2-DevKitM, symbol PCM_Espressif:ESP32-S2-DevKitM
Connections:
- net +3V3: now also U2.1 (3V3)
- net +5V: now also U2.20 (5V0)
- net ENVPIR_DIN: now also U2.16 (GPIO14/TOUCH14/ADC2_CH3/FSPIWP/FSPIDQS)
- net ENV_SCL: now also U2.28 (GPIO34)
- net ENV_SDA: now also U2.29 (GPIO35)
- net GND: now also U2.21 (GND), U2.42 (GND)
- net PIR_SCL: now also U2.13 (GPIO11/TOUCH11/ADC2_CH0/FSPID/FSPIIO5)
- net PIR_SDA: now also U2.12 (GPIO10/TOUCH10/ADC1_CH9/FSPICS0/FSPIIO4)
Other:
- note added: "2024-06-14"
- note removed: "2021-12-03"
- moved on the sheet: J1, J12, J13, J2, J3, J4, J5, J6, J7, R1, R2
