File: main_board/main_board.kicad_pcb (KiCad board)
At the start: 2 copper layers, 43.2 x 59.1 mm, 12 parts, among them J1 5V IN, J12 I2C ENV, J13 ENVPIR, J2 3.3V IN, J3 I2C PIR, J4 3.3V OUT, J5 3.3V OUT, U1 ESP32-S2-Saola-1

Commit message: Update to v0.5
Parts:
- removed U1: ESP32-S2-Saola-1, miro-v04:ESP32-S2-Saola-1
- added REF**: MountingHole_3.2mm_M3_DIN965_Pad, MountingHole:MountingHole_3.2mm_M3_DIN965_Pad, F.Cu at (173.5, 58.0)
- added REF**: MountingHole_3.2mm_M3_DIN965_Pad, MountingHole:MountingHole_3.2mm_M3_DIN965_Pad, F.Cu at (134.0, 94.0)
- added REF**: MountingHole_3.2mm_M3_DIN965_Pad, MountingHole:MountingHole_3.2mm_M3_DIN965_Pad, F.Cu at (173.5, 109.0)
- added U2: ESP32-S2-DevKitM, PCM_Espressif:ESP32-S2-DevKitM, F.Cu at (144.8, 57.1)
- moved LUX 34.8 mm to (173.5, 76.6), turned to 0 degrees
- moved T&H 26.0 mm to (173.5, 93.6), turned to 0 degrees
- moved J3 2.17 mm to (132.7, 81.5)
- moved R1 1.53 mm to (139.7, 89.5)
Routing:
- net /ENV_SCL: track 52.6 -> 63.3 mm, vias 2 -> 1
- net /PIR_SCL: track 14.1 -> 5.43 mm
- net /ENV_SDA: track 67.5 -> 75.4 mm, vias 4 -> 0
- net /PIR_SDA: track 15.4 -> 9.17 mm
- net +3V3: track 159.8 -> 154.7 mm
- net /ENVPIR_DIN: track 13.8 -> 13.0 mm
- net GND: vias 56 -> 67
Other:
- board size 43.2 x 59.1 mm -> 48.6 x 59.1 mm

Commit message: Some fixes and v0.5 labels
Routing:
- net /PIR_SCL: track 5.43 -> 13.4 mm
- net /PIR_SDA: track 9.17 -> 15.6 mm
- net GND: vias 67 -> 65
Other:
- board text added: "MIROSLAV v0.5 - Main board"
- board text removed: "MIROSLAV v0.4 - Main board"
Changed lines of the file:
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@@
 		(layer "Edge.Cuts")
 	)
-	(gr_text "MIROSLAV v0.4 - Main board"
+	(gr_text "MIROSLAV v0.5 - Main board"
 		(at 151.13 82.296 90)
 		(layer "B.SilkS")
@@
 	)
 	(via
-		(at 135.89 85.725)
+		(at 136.5 84.5)
 		(size 0.8)
 		(drill 0.4)
@@
 	)
 	(via
-		(at 134.62 81.28)
-		(size 0.8)
-		(drill 0.4)
-		(layers "F.Cu" "B.Cu")
-		(net 2)
-	)
-	(via
 		(at 160.655 107.95)
 		(size 0.8)
@@
 	(via
 		(at 165.1 69.215)
-		(size 0.8)
-		(drill 0.4)
-		(layers "F.Cu" "B.Cu")
-		(net 2)
-	)
-	(via
-		(at 138.43 85.725)
 		(size 0.8)
 		(drill 0.4)
@@
 	)
 	(segment
+		(start 137.1 91.1)
+		(end 136 90)
+		(width 0.5)
+		(layer "F.Cu")
+		(net 3)
+	)
+	(segment
 		(start 139.7 75.565)
 		(end 137.382498 73.247498)
@@
 	)
 	(segment
-		(start 138.6 90)
-		(end 130.175 90)
-		(width 0.5)
-		(layer "F.Cu")
-		(net 3)
-	)
-	(segment
 		(start 136.429998 74.199998)
 		(end 137.382498 73.247498)
@@
 	)
 	(segment
+		(start 136 90)
+		(end 130.175 90)
+		(width 0.5)
+		(layer "F.Cu")
+		(net 3)
+	)
+	(segment
+		(start 139.7 91.1)
+		(end 137.1 91.1)
+		(width 0.5)
+		(layer "F.Cu")
+		(net 3)
+	)
+	(segment
 		(start 137.890002 72.739994)
 		(end 137.890002 67.214998)
@@
 	)
 	(segment
-		(start 139.7 91.1)
-		(end 138.6 90)
-		(width 0.5)
-		(layer "F.Cu")
-		(net 3)
-	)
-	(segment
 		(start 130.175 90)
 		(end 130.175 77.47)
@@
 	)
 	(segment
-		(start 138.919999 83.674999)
-		(end 138.919999 82.060001)
+		(start 139.7 84.455)
+		(end 139.7 81.28)
+		(width 0.5)
+		(layer "F.Cu")
+		(net 4)
+	)
+	(segment
+		(start 132.715 81.5)
+		(end 139.48 81.5)
 		(width 0.5)
 		(layer "F.Cu")
@@
 	)
 	(segment
-		(start 138.919999 83.674999)
-		(end 140.33772 85.09272)
+		(start 140.33772 85.09272)
+		(end 139.7 84.455)
 		(width 0.5)
 		(layer "F.Cu")
@@
 	)
 	(segment
-		(start 138.919999 82.060001)
+		(start 139.48 81.5)
 		(end 139.7 81.28)
 		(width 0.5)
@@
 	)
 	(segment
-		(start 144.41 88)
-		(end 144.78 87.63)
+		(start 139.7 88)
+		(end 136.25 88)
+		(width 0.5)
+		(layer "F.Cu")
+		(net 5)
+	)
+	(segment
+		(start 133.849999 85.599999)
+		(end 132.715 85.599999)
+		(width 0.5)
+		(layer "F.Cu")
+		(net 5)
+	)
+	(segment
+		(start 136.25 88)
+		(end 133.849999 85.599999)
+		(width 0.5)
+		(layer "F.Cu")
+		(net 5)
+	)
+	(segment
+		(start 140.07 87.63)
+		(end 139.7 88)
 		(width 0.5)
 		(layer "F.Cu")
@@
 	)
 	(segment
-		(start 139.7 88)
-		(end 144.41 88)
-		(width 0.5)
-		(layer "F.Cu")
+		(start 144.78 87.63)
+		(end 140.07 87.63)
+		(width 0.5)
+		(layer "F.Cu")
