File: power_board/power_board.kicad_sch (KiCad schematic)
At the start: 30 parts, among them J1 PWR IN, J2 PWR IN, J3 MBOARD, J4 SBOARD

Commit message: Set proper revision date on POWERBOARD
Other:
- note added: "2023-06-14"
- note removed: "2021-12-08"
Changed lines of the file:
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@@
 		)
 	)
-	(text "2021-12-08"
+	(text "2023-06-14"
 		(exclude_from_sim no)
 		(at 207.01 194.31 0)
