File: power_board/power_board.kicad_pcb (KiCad board)
At the start: 2 copper layers, 20.6 x 99.1 mm, 28 parts, among them J3 MBOARD, J4 SBOARD

Commit message: Update to v0.5
Parts:
- added REF**: MountingHole_3.2mm_M3_DIN965_Pad, MountingHole:MountingHole_3.2mm_M3_DIN965_Pad, F.Cu at (105.0, 111.0)
- added REF**: MountingHole_3.2mm_M3_DIN965_Pad, MountingHole:MountingHole_3.2mm_M3_DIN965_Pad, F.Cu at (105.0, 42.8)
- moved PIR12 3.05 mm to (111.0, 29.1)
- moved PIR13 3.05 mm to (111.0, 36.1)
- moved PIR14 3.05 mm to (111.0, 43.1)
- moved PIR15 3.05 mm to (111.0, 50.0)
- moved PIR16 3.05 mm to (111.0, 57.0)
- moved PIR18 3.05 mm to (111.0, 71.0)
- moved PIR19 3.05 mm to (111.0, 78.0)
- moved PIR20 3.05 mm to (111.0, 85.0)
- moved PIR21 3.05 mm to (111.0, 92.0)
- moved PIR22 3.05 mm to (111.0, 98.9)
- moved PIR23 3.05 mm to (111.0, 105.9)
- moved PIR24 3.05 mm to (111.0, 112.9)
- moved PIR17 3.05 mm to (111.0, 64.0)
Other:
- board size 20.6 x 99.1 mm -> 23.8 x 99.1 mm
Changed lines of the file:
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@@
 	(footprint "miro-v04:TE_HDI_2_horiz_altsilk"
 		(layer "F.Cu")
-		(at 107.95 50.164999 90)
+		(at 111 50.044998 90)
 		(property "Reference" "PIR15"
 			(at 1.016 4.826 90)
@@
 	(footprint "miro-v04:TE_HDI_2_horiz_altsilk"
 		(layer "F.Cu")
-		(at 107.95 71.12 90)
+		(at 111 70.999999 90)
 		(property "Reference" "PIR18"
 			(at 1.016 4.826 90)
@@
 	(footprint "miro-v04:TE_HDI_2_horiz_altsilk"
 		(layer "F.Cu")
-		(at 107.95 99.06 90)
+		(at 111 98.939999 90)
 		(property "Reference" "PIR22"
 			(at 1.016 4.826 90)
@@
 	(footprint "miro-v04:TE_HDI_2_horiz_altsilk"
 		(layer "F.Cu")
-		(at 107.95 85.09 90)
+		(at 111 84.969999 90)
 		(property "Reference" "PIR20"
 			(at 1.016 4.826 90)
@@
 	(footprint "miro-v04:TE_HDI_2_horiz_altsilk"
 		(layer "F.Cu")
-		(at 107.95 36.195 90)
+		(at 111 36.074999 90)
 		(property "Reference" "PIR13"
 			(at 1.016 4.826 90)
@@
 	(footprint "miro-v04:TE_HDI_2_horiz_altsilk"
 		(layer "F.Cu")
-		(at 107.95 78.104999 90)
+		(at 111 77.984998 90)
 		(property "Reference" "PIR19"
 			(at 1.016 4.826 90)
@@
 	(footprint "miro-v04:TE_HDI_2_horiz_altsilk"
 		(layer "F.Cu")
-		(at 107.95 92.075 90)
+		(at 111 91.954999 90)
 		(property "Reference" "PIR21"
 			(at 1.016 4.826 90)
@@
 	(footprint "miro-v04:TE_HDI_2_horiz_altsilk"
 		(layer "F.Cu")
-		(at 107.95 57.15 90)
+		(at 111 57.029999 90)
 		(property "Reference" "PIR16"
 			(at 1.016 4.826 90)
@@
 	(footprint "miro-v04:TE_HDI_2_horiz_altsilk"
 		(layer "F.Cu")
-		(at 107.95 113.029999 90)
+		(at 111 112.909998 90)
 		(property "Reference" "PIR24"
 			(at -3.175001 3.429 0)
@@
 	(footprint "miro-v04:TE_HDI_2_horiz_altsilk"
 		(layer "F.Cu")
-		(at 107.95 43.18 90)
+		(at 111 43.059999 90)
 		(property "Reference" "PIR14"
 			(at 1.016 4.826 90)
@@
 	(footprint "miro-v04:TE_HDI_2_horiz_altsilk"
 		(layer "F.Cu")
-		(at 107.95 64.134999 90)
+		(at 111 64.014998 90)
 		(property "Reference" "PIR17"
 			(at 1.016 4.826 90)
@@
 	(footprint "miro-v04:TE_HDI_2_horiz_altsilk"
 		(layer "F.Cu")
-		(at 107.95 106.045 90)
+		(at 111 105.924999 90)
 		(property "Reference" "PIR23"
 			(at 1.016 4.826 90)
@@
 	(footprint "miro-v04:TE_HDI_2_horiz_altsilk"
 		(layer "F.Cu")
-		(at 107.95 29.21 90)
+		(at 111 29.089999 90)
 		(property "Reference" "PIR12"
 			(at 1.016 4.826 90)
@@
 		)
 	)
+	(footprint "MountingHole:MountingHole_3.2mm_M3_DIN965_Pad"
+		(layer "F.Cu")
+		(at 105 111)
+		(descr "Mounting Hole 3.2mm, M3, DIN965")
+		(tags "mounting hole 3.2mm m3 din965")
+		(property "Reference" "REF**"
+			(at 0 -3.8 0)
+			(layer "F.SilkS")
+			(effects
+				(font
+					(size 1 1)
+					(thickness 0.15)
+				)
+			)
+		)
+		(property "Value" "MountingHole_3.2mm_M3_DIN965_Pad"
+			(at 0 3.8 0)
+			(layer "F.Fab")
+			(effects
+				(font
+					(size 1 1)
+					(thickness 0.15)
+				)
+			)
+		)
+		(property "Footprint" "MountingHole:MountingHole_3.2mm_M3_DIN965_Pad"
+			(at 0 0 0)
+			(unlocked yes)
+			(layer "F.Fab")
+			(hide yes)
+			(effects
+				(font
+					(size 1.27 1.27)
+					(thickness 0.15)
+				)
+			)
+		)
+		(property "Datasheet" ""
+			(at 0 0 0)
+			(unlocked yes)
+			(layer "F.Fab")
+			(hide yes)
+			(effects
+				(font
+					(size 1.27 1.27)
+					(thickness 0.15)
+				)
+			)
+		)
+		(property "Description" ""
+			(at 0 0 0)
+			(unlocked yes)
+			(layer "F.Fab")
+			(hide yes)
+			(effects
+				(font
+					(size 1.27 1.27)
+					(thickness 0.15)
+				)
+			)
+		)
+		(attr exclude_from_pos_files exclude_from_bom)
+		(fp_circle
+			(center 0 0)
+			(end 2.8 0)
+			(stroke
+				(width 0.15)
+				(type solid)
+			)
+			(fill none)
+			(layer "Cmts.User")
+		)
+		(fp_circle
+			(center 0 0)
+			(end 3.05 0)
+			(stroke
+				(width 0.05)
+				(type solid)
+			)
+			(fill none)
+			(layer "F.CrtYd")
+		)
+		(fp_text user "${REFERENCE}"
+			(at 0 0 0)
+			(layer "F.Fab")
+			(effects
+				(font
+					(size 1 1)
+					(thickness 0.15)
+				)
+			)
+		)
+		(pad "1" thru_hole circle
+			(at 0 0)
+			(size 5.6 5.6)
+			(drill 3.2)
+			(layers "*.Cu" "*.Mask")
+			(remove_unused_layers no)
+		)
+	)
+	(footprint "MountingHole:MountingHole_3.2mm_M3_DIN965_Pad"
+		(layer "F.Cu")
+		(at 105 42.75)
+		(descr "Mounting Hole 3.2mm, M3, DIN965")
+		(tags "mounting hole 3.2mm m3 din965")
+		(property "Reference" "REF**"
+			(at 0 -3.8 0)
+			(layer "F.SilkS")
+			(effects
+				(font
+					(size 1 1)
+					(thickness 0.15)
+				)
+			)
+		)
+		(property "Value" "MountingHole_3.2mm_M3_DIN965_Pad"
+			(at 0 3.8 0)
+			(layer "F.Fab")
+			(effects
+				(font
+					(size 1 1)
+					(thickness 0.15)
+				)
+			)
+		)
+		(property "Footprint" "MountingHole:MountingHole_3.2mm_M3_DIN965_Pad"
+			(at 0 0 0)
+			(unlocked yes)
+			(layer "F.Fab")
+			(hide yes)
+			(effects
+				(font
+					(size 1.27 1.27)
+					(thickness 0.15)
+				)
+			)
+		)
+		(property "Datasheet" ""
+			(at 0 0 0)
+			(unlocked yes)
+			(layer "F.Fab")
+			(hide yes)
+			(effects
+				(font
+					(size 1.27 1.27)
+					(thickness 0.15)
+				)
+			)
+		)
+		(property "Description" ""
+			(at 0 0 0)
+			(unlocked yes)
+			(layer "F.Fab")
+			(hide yes)
+			(effects
+				(font
+					(size 1.27 1.27)
+					(thickness 0.15)
+				)
+			)
+		)
+		(attr exclude_from_pos_files exclude_from_bom)
+		(fp_circle
+			(center 0 0)
+			(end 2.8 0)
+			(stroke
+				(width 0.15)
+				(type solid)
+			)
+			(fill none)
+			(layer "Cmts.User")
+		)
+		(fp_circle
+			(center 0 0)
+			(end 3.05 0)
+			(stroke
+				(width 0.05)
+				(type solid)
+			)
+			(fill none)
+			(layer "F.CrtYd")
+		)
+		(fp_text user "${REFERENCE}"
+			(at 0 0 0)
+			(layer "F.Fab")
+			(effects
+				(font
+					(size 1 1)
+					(thickness 0.15)
+				)
+			)
+		)
+		(pad "1" thru_hole circle
+			(at 0 0)
+			(size 5.6 5.6)
+			(drill 3.2)
+			(layers "*.Cu" "*.Mask")
+			(remove_unused_layers no)
+		)
+	)
 	(gr_line
 		(start 104.775 105.41)
@@
 	)
 	(gr_line
-		(start 113.792 24.638)
+		(start 117 24.638)
 		(end 93.218 24.638)
 		(stroke
@@
 	)
 	(gr_line
-		(start 113.792 123.698)
-		(end 113.792 24.638)
+		(start 117 123.698)
+		(end 117 24.638)
 		(stroke
 			(width 0.1)
@@
 	(gr_line
 		(start 93.218 123.698)
-		(end 113.792 123.698)
+		(end 117 123.698)
 		(stroke
 			(width 0.1)
@@
 		(polygon
 			(pts
-				(xy 113.792 123.698) (xy 93.218 123.698) (xy 93.218 24.638) (xy 113.792 24.638)
+				(xy 117 123.698) (xy 93.218 123.698) (xy 93.218 24.638) (xy 117 24.638)
 			)
 		)
@@
 		(polygon
 			(pts
-				(xy 113.792 123.698) (xy 93.218 123.698) (xy 93.218 24.638) (xy 113.792 24.638)
+				(xy 117 123.698) (xy 93.218 123.698) (xy 93.218 24.638) (xy 117 24.638)
 			)
 		)

Commit message: Some fixes and v0.5 labels
Other:
- board text added: "MIROSLAV v0.5 - Power distribution board"
- board text removed: "MIROSLAV v0.4 - Power distribution board"
Changed lines of the file:
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@@
 		(layer "Edge.Cuts")
 	)
-	(gr_text "MIROSLAV v0.4 - Power distribution board"
-		(at 103.505 69.215 -90)
+	(gr_text "MIROSLAV v0.5 - Power distribution board"
+		(at 103.5 72.5 270)
 		(layer "B.SilkS")
 		(effects
