File: serialization_board/serialization_board.kicad_pcb (KiCad board)
At the start: 2 copper layers, 24.9 x 74.2 mm, 24 parts, among them J1 3.3V IN, J2 I2C, J3 INT, J6 3.3V stack, J7 I2C stack, U1 MCP_X

Commit message: Some fixes and v0.5 labels
Parts:
- I2C stack: moved to B.Cu
- J6: moved to B.Cu
- turned I2C stack to 0 degrees
- turned J6 to 180 degrees
Other:
- board text added: "I2C stack"
- board text added: "MIROSLAV v0.4.1 - Serialization board"
- board text added: "PWR st."
- board text removed: "MIROSLAV v0.4 - Serialization board"
